File: power/power.sch (KiCad schematic (older format))
At the start: 38 parts, among them Q1 TIP120, U1 LevelShifter

Commit message: main changes
Parts:
- removed C_MD_L1, C_MD_L2: 100uF, Capacitor_THT:CP_Radial_D5.0mm_P2.50mm, symbol Device:CP
- removed Con_MainBoard2PowerBoard1: Conn_01x09_Female, Connector_PinSocket_2.54mm:PinSocket_1x11_P2.54mm_Vertical, symbol Connector:Conn_01x11_Female
- removed Con_Motor_L1, Con_Motor_R1, Display_Connector1: Conn_01x04, Connector_JST:JST_XH_B4B-XH-A_1x04_P2.50mm_Vertical, symbol Connector_Generic:Conn_01x04
- removed MD_L1, MD_R1: Pololu_Breakout_A4988, Module:Pololu_Breakout-16_15.2x20.3mm, symbol Driver_Motor:Pololu_Breakout_A4988
- removed MicroController1: IZOKEEProMini, CustomFootprints:Arduino_Pro_Mini_Socket_IZOKEE, symbol Custom:IZOKEEProMini
- removed RPi_Connector1: Conn_01x05, Connector_JST:JST_XH_B5B-XH-A_1x05_P2.50mm_Vertical, symbol Connector_Generic:Conn_01x05
- removed U1: LevelShifter, CustomFootprints:LevelShifterBreakoutBoard, symbol Custom:LevelShifter
- Switch_Connector1: footprint Connector_JST:JST_XH_B4B-XH-A_1x04_P2.50mm_Vertical -> Connector_JST:JST_XH_B2B-XH-A_1x02_P2.50mm_Vertical; symbol Connector_Generic:Conn_01x04 -> Connector_Generic:Conn_01x02
Connections:
- net labels removed: +3.3V, Dir_L, Dir_R, Enable_Steppers, I2C_SCL, I2C_SDA, MS1_L, MS1_R, MS2_L, MS2_R, MS3_L, MS3_R, PCheck, PowerIN, Step_L, Step_R
- wire segments 70 -> 63
Other:
- note removed: "Main Board"
