File: mainboard/_autosave-main.sch (KiCad schematic (older format))
At the start: 38 parts, among them Q1 TIP120, U1 LevelShifter

Commit message: merge boards
Connections:
- net PCheck is gone; now on net P_Check: MicroController1.18 (A7)
- net PowerIN is gone; now on net P_IN: MicroController1.17 (D13/SCK)
Changed lines of the file:
@@
 $EndDescr
 Text GLabel 2200 2600 3    40   Input ~ 0
-PCheck
+P_Check
 Text GLabel 1700 1700 0    40   Input ~ 0
-PowerIN
+P_IN
 Wire Wire Line
 	1700 1600 1250 1600

Commit message: first prototype
Parts:
- removed C1: 1uF, Capacitor_THT:CP_Radial_D5.0mm_P2.50mm, symbol Device:CP
- removed CellVoltageOpAmp1: LM358, Package_DIP:DIP-8_W7.62mm_Socket, symbol Amplifier_Operational:LM358
- removed R_Cell1_Vdiv_A1: 33K, Resistor_THT:R_Axial_DIN0207_L6.3mm_D2.5mm_P7.62mm_Horizontal, symbol Device:R
- removed R_Cell1_Vdiv_B1: 100K, Resistor_THT:R_Axial_DIN0207_L6.3mm_D2.5mm_P2.54mm_Vertical, symbol Device:R
- removed R_V_Cell2_1, R_V_Cell2_2, R_V_Cell3_2: 47K, Resistor_THT:R_Axial_DIN0207_L6.3mm_D2.5mm_P2.54mm_Vertical, symbol Device:R
- removed R_V_Cell2_3, R_V_Cell2_4, R_V_Cell3_3, R_V_Cell3_4: 33K, Resistor_THT:R_Axial_DIN0207_L6.3mm_D2.5mm_P2.54mm_Vertical, symbol Device:R
- removed R_V_Cell3_1: 47K, Resistor_THT:R_Axial_DIN0207_L6.3mm_D2.5mm_P5.08mm_Vertical, symbol Device:R
- added Diode2, Diode3: D, Diode_THT:D_T-1_P5.08mm_Horizontal, symbol Device:D
- added R1: ?, Resistor_THT:R_Axial_DIN0207_L6.3mm_D2.5mm_P2.54mm_Vertical, symbol Device:R
- added RV2: R_POT3Bat, Potentiometer_THT:Potentiometer_Bourns_3296W_Vertical, symbol Device:R_POT_TRIM
- added RV3: R_POT2, Potentiometer_THT:Potentiometer_Bourns_3296W_Vertical, symbol Device:R_POT_TRIM
- added RV4: R_POT1, Potentiometer_THT:Potentiometer_Bourns_3296W_Vertical, symbol Device:R_POT_TRIM
- MicroController1: footprint CustomFootprints:Arduino_Pro_Mini_Socket_IZOKEE -> CustomFootprints:Arduino_Pro_Mini_Socket_IZOKEE_no_programming
- renumbered Diode1 to Diode1sw1
Connections:
- net +3V3: no longer Con_Switch1.3 (Pin_3)
- net +BATT: now also RV3.3
- net BATT_Cell_1_2: now also Diode3.2 (A)
- net BATT_Cell_2_3: now also Diode2.2 (A)
- net GND: now also Con_Switch1.3 (Pin_3), RV2.1, RV3.1, RV4.1
- net op2: now also RV2.2
- net op3: now also RV3.2
- net op4: now also RV4.2
- net at Diode1sw1.1 (K), RV1.3, R_T1.1: now also R1.2; no longer Switch_Connector1.2 (Pin_2)
- new net: R1.1, Switch_Connector1.2 (Pin_2)
- new net: Diode2.1 (K), RV2.3
- new net: Diode3.1 (K), RV4.3
